Commit message: Agregando archivos desde otras carpetas

File: src/KUKA_16/kr16_gazebo/urdf/gazebo.xacro (robot description, xacro)
@@ -1,5 +1,5 @@
 <?xml version="1.0" ?>
 <robot name="kuka_kr16_gazebo" xmlns:xacro="http://wiki.ros.org/xacro">
-  <!-- KR10 -->
+  <!-- KR16 -->
   <xacro:include filename="$(find kr16_gazebo)/urdf/gazebo_transmission.xacro"/>
   <xacro:kuka_kr16_robot prefix=""/>
@@ -11,189 +11,3 @@
     <origin xyz="0.0 0.0 0.0" rpy="0.0 0.0 0.0" />
   </joint>
-  <!-- camera plugin -->
-  <link name="camera">
-    <collision>
-      <origin rpy="0 0 0" xyz="0 0 0"/>
-      <geometry>
-        <box size="0.1 0.7 0.7"/>
-      </geometry>
-    </collision>
-    <visual>
-      <origin rpy="0 0 0" xyz="0 0 0"/>
-      <geometry>
-        <box size="0.1 0.7 0.7"/>
-      </geometry>
-      <material name="grey"/>
-    </visual>
-    <inertial>
-      <mass value="0.1"/>
-      <origin rpy="0 0 0" xyz="0 0 0"/>
-      <box_inertia m="0.1" x="0.1" y="0.7" z="0.7"/>
-      <inertia ixx="1e-6" ixy="0" ixz="0" iyy="1e-6" iyz="0" izz="1e-6"/>
-    </inertial>
-  </link>
-  <joint name="camera_optical_joint" type="fixed">
-    <origin rpy="-1.5708 0 -1.5708" xyz="0 0 0"/>
-    <parent link="camera"/>
-    <child link="camera_frame_optical"/>
-  </joint>
-  <link name="camera_frame_optical"/>
-  <joint name="camera_joint" type="fixed">
-    <axis xyz="0 0 0"/>
-    <origin rpy="0 1.5708 0" xyz="0.5 0 2.0"/>
-    <parent link="base_link"/>
-    <child link="camera"/>
-  </joint>
-  <!-- depth camera -->
-  <gazebo reference="camera">
-    <sensor name="camera1" type="depth">
-      <update_rate>20</update_rate>
-      <camera>
-        <horizontal_fov>1.2</horizontal_fov>
-        <image>
-          <width>640</width>
-          <!--640-->
-          <height>480</height>
-          <!--480-->
-          <format>R8G8B8</format>
-        </image>
-        <clip>
-          <near>0.05</near>
-          <far>30</far>
-        </clip>
-      </camera>
-      <plugin filename="libgazebo_ros_openni_kinect.so" name="camera_controller">
-        <baseline>0.2</baseline>
-        <alwaysOn>false</alwaysOn>
-        <updateRate>1.0</updateRate>
-        <cameraName>camera1</cameraName>
-        <imageTopicName>/camera1/color/image_raw</imageTopicName>
-        <cameraInfoTopicName>/camera1/color/camera_info</cameraInfoTopicName>
-        <depthImageTopicName>/camera1/depth/image_raw</depthImageTopicName>
-        <depthImageInfoTopicName>/camera1/depth/camera_info</depthImageInfoTopicName>
-        <pointCloudTopicName>/camera1/depth/points</pointCloudTopicName>
-        <frameName>camera_frame_optical</frameName>
-        <pointCloudCutoff>0.5</pointCloudCutoff>
-        <pointCloudCutoffMax>3.0</pointCloudCutoffMax>
-        <distortionK1>0.00000001</distortionK1>
-        <distortionK2>0.00000001</distortionK2>
-        <distortionK3>0.00000001</distortionK3>
-        <distortionT1>0.00000001</distortionT1>
-        <distortionT2>0.00000001</distortionT2>
-        <CxPrime>0</CxPrime>
-        <Cx>0</Cx>
-        <Cy>0</Cy>
-        <focalLength>0</focalLength>
-        <hackBaseline>0</hackBaseline>
-      </plugin>
-    </sensor>
-  </gazebo>
-  <!-- caja 1 plugin -->
-  <link name="caja1">
-    <collision>
-      <origin rpy="0 0 0" xyz="0 0 0"/>
-      <geometry>
-        <box size="0.2 0.3 0.1"/>
-      </geometry>
-    </collision>
-    <visual>
-      <origin rpy="0 0 0" xyz="0 0 0"/>
-      <geometry>
-        <box size="0.2 0.3 0.1"/>
-      </geometry>
-      <material name="grey">
-        <color rgba="0.5 0.5 0.5 1"/>
-      </material>
-    </visual>
-    <inertial>
-      <mass value="10"/>
-      <origin rpy="0 0 0" xyz="0 0 0"/>
-      <box_inertia m="10" x="0.2" y="0.3" z="0.1"/>
-      <inertia ixx="1e-6" ixy="0" ixz="0" iyy="1e-6" iyz="0" izz="1e-6"/>
-    </inertial>
-  </link>
-  <joint name="caja1_optical_joint" type="fixed">
-    <origin rpy="-1.5708 0 -1.5708" xyz="0 0 0"/>
-    <parent link="caja1"/>
-    <child link="caja_optical"/>
-  </joint>
-  <link name="caja_optical"/>
-  <joint name="caja_joint" type="fixed">
-    <axis xyz="0 0 0"/>
-    <origin rpy="0 1.5708 0" xyz="1.5 0 0.1"/>
-    <parent link="base_link"/>
-    <child link="caja1"/>
-  </joint>
-   <!-- caja 2 plugin -->
-  <link name="caja2">
-    <collision>
-      <origin rpy="0 0 0" xyz="0 0 0"/>
-      <geometry>
-        <box size="0.2 0.3 0.05"/>
-      </geometry>
-    </collision>
-    <visual>
-      <origin rpy="0 0 0" xyz="0 0 0"/>
-      <geometry>
-        <box size="0.2 0.3 0.05"/>
-      </geometry>
-      <material name="grey">
-        <color rgba="0.5 0.5 0.5 1"/>
-      </material>
-    </visual>
-    <inertial>
-      <mass value="10"/>
-      <origin rpy="0 0 0" xyz="0 0 0"/>
-      <box_inertia m="10" x="0.2" y="0.3" z="0.05"/>
-      <inertia ixx="1e-6" ixy="0" ixz="0" iyy="1e-6" iyz="0" izz="1e-6"/>
-    </inertial>
-  </link>
-  <joint name="caja2_optical_joint" type="fixed">
-    <origin rpy="-1.5708 0 -1.5708" xyz="0 0 0"/>
-    <parent link="caja2"/>
-    <child link="caja2_optical"/>
-  </joint>
-  <link name="caja2_optical"/>
-  <joint name="caja2_joint" type="fixed">
-    <axis xyz="0 0 0"/>
-    <origin rpy="0 1.5708 0" xyz="1 -1 0.1"/>
-    <parent link="base_link"/>
-    <child link="caja2"/>
-  </joint>
-   <!-- caja 3 plugin -->
-  <link name="caja3">
-    <collision>
-      <origin rpy="0 0 0" xyz="0 0 0"/>
-      <geometry>
-        <box size="0.2 0.3 0.03"/>
-      </geometry>
-    </collision>
-    <visual>
-      <origin rpy="0 0 0" xyz="0 0 0"/>
-      <geometry>
-        <box size="0.2 0.3 0.03"/>
-      </geometry>
-      <material name="grey">
-        <color rgba="0.5 0.5 0.5 1"/>
-      </material>
-    </visual>
-    <inertial>
-      <mass value="10"/>
-      <origin rpy="0 0 0" xyz="0 0 0"/>
-      <box_inertia m="10" x="0.2" y="0.3" z="0.03"/>
-      <inertia ixx="1e-6" ixy="0" ixz="0" iyy="1e-6" iyz="0" izz="1e-6"/>
-    </inertial>
-  </link>
-  <joint name="caja3_optical_joint" type="fixed">
-    <origin rpy="-1.5708 0 -1.5708" xyz="0 0 0"/>
-    <parent link="caja3"/>
-    <child link="caja3_optical"/>
-  </joint>
-  <link name="caja3_optical"/>
-  <joint name="caja3_joint" type="fixed">
-    <axis xyz="0 0 0"/>
-    <origin rpy="0 1.5708 0" xyz="1 1 0.1"/>
-    <parent link="base_link"/>
-    <child link="caja3"/>
-  </joint>
 </robot>

File: src/KUKA_16/kr16_gazebo/urdf/gazebo_2f.xacro (robot description, xacro)
@@ -1,5 +1,4 @@
 <?xml version="1.0" ?>
 <robot name="kuka_kr16_gripper" xmlns:xacro="http://ros.org/wiki/xacro">
-  <xacro:include filename="$(find kr16_gazebo)/urdf/gazebo.xacro"/>
   <xacro:include filename="$(find robotiq_2f_85_description)/urdf/robotiq_2F_85.xacro"/>
   <xacro:property name="PI" value="3.1415926535897931"/>
@@ -7,5 +6,5 @@
     <parent link="tool0"/>
     <child link="coupling_link"/>
-    <origin rpy="0 0 0" xyz="0 0 -0.003"/>
+    <origin rpy="0 0 0" xyz="0 0 0.01"/>
   </joint>
   <xacro:include filename="$(find kr16_gazebo)/urdf/transmission_2f.xacro"/>
